Commit message: setup robot for simulation. add launch file

File: dev_ws/src/warehouse_robot/description/robot_core.xacro (robot description, xacro)
@@ -45,4 +45,7 @@
         </xacro:inertial_box>
     </link>
+    <gazebo reference="chassis">
+        <material>Gazebo/White</material>
+    </gazebo>
     <!-- LEFT WHEEL LINK-->
     <joint name="left_wheel_joint" type="continuous">
@@ -69,4 +72,7 @@
         </xacro:inertial_cylinder>
     </link>
+    <gazebo reference="left_wheel">
+        <material>Gazebo/Blue</material>
+    </gazebo>
     <!-- RIGHT WHEEL LINK-->
     <joint name="right_wheel_joint" type="continuous">
@@ -93,4 +99,7 @@
         </xacro:inertial_cylinder>
     </link>
+    <gazebo reference="right_wheel">
+        <material>Gazebo/Blue</material>
+    </gazebo>
     <!-- CASTER WHEEL LINK-->
     <joint name="caster_wheel_joint" type="fixed">
@@ -115,3 +124,8 @@
         </xacro:inertial_sphere>
     </link>
+    <gazebo reference="caster_wheel">
+        <material>Gazebo/Black</material>
+        <mu1 value="0.001"/>
+        <mu2 value="0.001"/>
+    </gazebo>
 </robot>

Commit message: add warehouse model to gazebo. remove install and log from git

File: dev_ws/src/warehouse_robot/description/robot_core.xacro (robot description, xacro)
@@ -34,4 +34,12 @@
     <link name="base_link">
     </link>
+    <!-- BASE_FOOTPRINT LINK-->
+     <joint name="base_footprint_joint" type="fixed">
+        <parent link="base_link"/>
+        <child link="base_footprint"/>
+        <origin xyz="0 0 0" rpy="0 0 0"/>
+     </joint>
+     <link name="base_footprint">
+     </link>
     <!-- CHASSIS LINK-->
     <joint name="chassis_joint" type="fixed">
